File: board/board_revA.sch (EAGLE design)
At the start: 64 parts, among them IC1 MCP1703CB, IC2 STM32F042CX, IC3 MC1525TT, Q2 ULN2003AS, U1 HC_05, Y1 8Mhz

Commit message: [Board] Cleaning, WIP
Connections:
- new net VDD1: IC2.VDD1, IC2.VDD2
- net +3V3: now also IC2.VBAT
- net BOOT0: now also IC2.BOOT0
- net GND: now also IC2.VSS1, IC2.VSS2, IC2.VSSA
- net NRST: now also IC2.NRST
- net OSC_IN: now also IC2.PF0-OSC_IN
- net OSC_OUT: now also IC2.PF1-OSC_OUT
- net SWCLK: now also IC2.PA14-SWCLK
- net SWDAT: now also IC2.PA13-IROUT/SWDIO
- net VDDA: now also IC2.VDDA
Other:
- moved on the sheet: C3, R11, R12

Commit message: [Board] Working on schema
Parts:
- added JP2: (no value), SparkFun-Connectors:M04LOCK
Connections:
- new net BT_RST: U1.RST
- new net UART2_CTS: IC2.PA0-TIM2CH1ETR-ADC0/RTC_TAMP2/WKUP1, U1.RTS
- new net UART2_RTS: IC2.PA1-TIM2CH2/EVENTOUT-ADC1, U1.CTS
- new net UART3_RX: IC2.PB11-TIM2CH4/EVENTOUT, IC_KLINE.RXD@1, R2.1
- new net UART3_TX: IC2.PB10-TIM2CH3, IC_KLINE.TXD@4
- new net USB_DM: IC2.PA11-USART1CTS/TIM1CH4/EVENTOUT, JP2.2
- new net USB_DP: IC2.PA12-USART1RTS/TIM1ETR/EVENTOUT, JP2.3
- net +3V3: now also U1.3V3
- net +5V: now also JP2.4
- net GND: now also JP2.1, U1.GND, U1.GND1, U1.GND2
- net SPI2_MISO: now also IC2.PB14-TIM1CH2N
- net SPI2_MOSI: now also IC2.PB15-TIM1CH3N-RTCREFIN
- net SPI2_NSS: now also IC2.PB12-TIM1BKIN/EVENTOUT
- net SPI2_SCK: now also IC2.PB13-TIM1CH1N
- net UART2_RX: now also IC2.PA3-TIM2CH4-ADC3, U1.TX; no longer IC_KLINE.RXD@1, R2.1
- net UART2_TX: now also IC2.PA2-TIM2CH3-ADC2, U1.RX; no longer IC_KLINE.TXD@4
