File: board/board_revA.brd (EAGLE design)
At the start: 94 x 44.5 mm, 69 parts, among them IC1 MCP1703CB, IC2 STM32F042CX, IC3 MC1525TT, Q2 ULN2003AS, U1 HC_05, Y1 8Mhz

Commit message: [Board] Cleaning, WIP
Parts:
- moved C1 81.0 mm to (10.8, 41.9), turned to 180 degrees
- moved TP2 78.2 mm to (16.0, 42.2), flipped to the top
- moved D1 72.8 mm to (3.39, 32.8), flipped to the top
- moved S1 70.6 mm to (89.5, 12.2)
- moved IC_REG 68.8 mm to (22.8, 37.2), flipped to the top
- moved TP3 67.2 mm to (10.5, 39.2), flipped to the top
- moved R25 59.5 mm to (9.25, 31.0), flipped to the top
- moved C2 55.8 mm to (28.7, 34.9), flipped to the top
- moved CON_DBG 49.3 mm to (73.5, 5.50), flipped to the top
- moved Q2 44.3 mm to (17.0, 26.8), flipped to the top, turned to 180 degrees
- moved R26 44.1 mm to (22.8, 31.2), flipped to the top, turned to 0 degrees
- moved IC1 38.9 mm to (32.8, 31.8), flipped to the top
- moved D3 38.9 mm to (27.7, 8.08), flipped to the top
- moved R23 34.7 mm to (28.8, 24.5), flipped to the top
- moved R7 33.6 mm to (29.8, 11.7), flipped to the top
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Connections:
- new net VDD1: IC2.24, IC2.48
- net +3V3: now also IC2.1
- net BOOT0: now also IC2.44
- net GND: now also IC2.23, IC2.47, IC2.8
- net NRST: now also IC2.7
- net OSC_IN: now also IC2.5
- net OSC_OUT: now also IC2.6
- net SWCLK: now also IC2.37
- net SWDAT: now also IC2.34
- net VDDA: now also IC2.9
Other:
- board text removed: "ANALOG"
- board text removed: "CAN"
- board text removed: "K-LINE"
- board text removed: "POWER"
- board text removed: "RPM/SPD"

Commit message: [Board] Working on schema
Parts:
- added JP2: (no value), SparkFun-Connectors:1X04_LOCK
- moved U$6 36.0 mm to (54.0, 15.3)
- moved TP2 10.8 mm to (22.2, 33.5)
- moved TP3 8.19 mm to (3.50, 35.0)
- moved C6 7.50 mm to (59.5, 15.8), flipped to the top
- moved C1 4.32 mm to (15.2, 41.9), turned to 0 degrees
- moved IC_REG 1.82 mm to (22.2, 39.0)
- moved IC_EE 0.75 mm to (47.5, 10.0), turned to 0 degrees
- moved U1 0.25 mm to (80.2, 22.8)
- turned IC2 to 180 degrees
Connections:
- new net BT_RST: U1.11
- new net UART2_CTS: IC2.10, U1.4
- new net UART2_RTS: IC2.11, U1.3
- new net UART3_RX: IC2.22, IC_KLINE.1, R2.1
- new net UART3_TX: IC2.21, IC_KLINE.4
- new net USB_DM: IC2.32, JP2.2
- new net USB_DP: IC2.33, JP2.3
- net +3V3: now also U1.12
- net +5V: now also JP2.4
- net GND: now also JP2.1, U1.13, U1.21, U1.22
- net SPI2_MISO: now also IC2.27
- net SPI2_MOSI: now also IC2.28
- net SPI2_NSS: now also IC2.25
- net SPI2_SCK: now also IC2.26
- net UART2_RX: now also IC2.13, U1.1; no longer IC_KLINE.1, R2.1
- net UART2_TX: now also IC2.12, U1.2; no longer IC_KLINE.4
